Commit message: kansjek

File: urdf/robot_description.urdf.xacro (robot description, xacro)
@@ -1,7 +1,10 @@
 <?xml version="1.0"?>
 <robot name="block" xmlns:xacro="http://www.ros.org/wiki/xacro">
+  <!-- Masseløs root for å unngå KDL-advarsel -->
+  <link name="DUMMY"/>
+  <!-- Kropp med masse/inerti -->
   <link name="block_link">
     <inertial>
-      <mass value="1.0"/>
+      <mass value="60"/>
       <origin xyz="0 0 0"/>
       <inertia ixx="0.01" iyy="0.01" izz="0.01" ixy="0" ixz="0" iyz="0"/>
@@ -17,12 +20,29 @@
     </collision>
   </link>
-  <link name="DUMMY"/>
+  <!-- Root = DUMMY -> block_link -->
   <joint name="dummy_to_block" type="fixed">
-    <parent link="block_link"/>
-    <child link="DUMMY"/>
+    <parent link="DUMMY"/>
+    <child  link="block_link"/>
     <origin xyz="0 0 0" rpy="0 0 0"/>
   </joint>
+  <!-- Link-spesifikke Gazebo-parametre -->
   <gazebo reference="block_link">
-    <mu1>0.5</mu1><mu2>0.5</mu2><kp>100000</kp><kd>1</kd>
+    <mu1>0.5</mu1>
+    <mu2>0.5</mu2>
+    <kp>100000</kp>
+    <kd>1</kd>
+  </gazebo>
+  <gazebo>
+    <plugin name="buoyancy" filename="libbuoyancy_plugin.so">
+      <fluid_density>1250</fluid_density>
+      <surface_z>0.0</surface_z>
+      <link name="block_link">
+        <waterplane_area>2</waterplane_area>
+        <height>0.4</height>
+        <linear_damping>5.0</linear_damping>
+        <angular_damping>1.0</angular_damping>
+        <k_righting>50.0</k_righting>
+      </link>
+    </plugin>
   </gazebo>
 </robot>

Commit message: VANNET FUNKER

File: urdf/robot_description.urdf.xacro (robot description, xacro)
@@ -6,7 +6,11 @@
   <link name="block_link">
     <inertial>
-      <mass value="60"/>
+      <mass value="30.0"/>
       <origin xyz="0 0 0"/>
-      <inertia ixx="0.01" iyy="0.01" izz="0.01" ixy="0" ixz="0" iyz="0"/>
+      <!-- Boks 1x0.4x0.2 m, m=80 kg, CoM i origo:
+           Ixx = 1/12*m*(0.4^2+0.2^2) = 1.3333
+           Iyy = 1/12*m*(1.0^2+0.2^2) = 6.9333
+           Izz = 1/12*m*(1.0^2+0.4^2) = 7.7333 -->
+      <inertia ixx="1.3333" iyy="6.9333" izz="7.7333" ixy="0" ixz="0" iyz="0"/>
     </inertial>
     <visual>
@@ -26,21 +30,19 @@
     <origin xyz="0 0 0" rpy="0 0 0"/>
   </joint>
-  <!-- Link-spesifikke Gazebo-parametre -->
-  <gazebo reference="block_link">
-    <mu1>0.5</mu1>
-    <mu2>0.5</mu2>
-    <kp>100000</kp>
-    <kd>1</kd>
-  </gazebo>
   <gazebo>
-    <plugin name="buoyancy" filename="libbuoyancy_plugin.so">
-      <fluid_density>1250</fluid_density>
+    <plugin name="buoyancy" filename="/home/rocotics/ros2_ws/install/buoyancy_plugin/lib/libbuoyancy_plugin.so">
+      <fluid_density>1025</fluid_density>
       <surface_z>0.0</surface_z>
-      <link name="block_link">
-        <waterplane_area>2</waterplane_area>
-        <height>0.4</height>
-        <linear_damping>5.0</linear_damping>
-        <angular_damping>1.0</angular_damping>
+      <link name="DUMMY">
+        <waterplane_area>0.4</waterplane_area>
+        <height>0.2</height>
+        <linear_damping>60.0</linear_damping>
+        <angular_damping>10.0</angular_damping>
         <k_righting>50.0</k_righting>
+        <cob>
+          <x>0</x>
+          <y>0</y>
+          <z>-0.05</z>
+        </cob>
       </link>
     </plugin>
