Commit message: ?

File: urdf/ele306baat.urdf.xacro (robot description, xacro)
@@ -1,40 +1,52 @@
-<?xml version='1.0' encoding='utf-8'?>
-<robot name="ele306baat">
-    <link name="base_link">
-        <inertial>
-            <origin xyz="-0.5552386532467776 0.19999999999999993 0.09853724397359867" rpy="0.0 0.0 0.0" />
-            <mass value="30" />
-            <inertia ixx="6.19751676834202" iyy="31.207900541600267" izz="34.91016063035846" ixy="-7.105427357601002e-15" iyz="-2.6645352591003757e-15" ixz="1.0508686428543967" />
-        </inertial>
-        <visual name="base_link_visual">
-            <origin xyz="0.0 0.0 0.0" rpy="0.0 0.0 0.0" />
-            <geometry>
-                <mesh filename="$(find usv_package)/meshes/base_link.stl" scale="0.001 0.001 0.001" />
-            </geometry>
-        </visual>
-        <collision name="base_link_collision">
-            <origin xyz="0.0 0.0 0.0" rpy="0.0 0.0 0.0" />
-            <geometry>
-                <mesh filename="$(find usv_package)/meshes/base_link.stl" scale="0.001 0.001 0.001" />
-            </geometry>
-        </collision>
-    </link>
-    <gazebo>
-        <plugin name="buoyancy" filename="/home/rocotics/ros2_ws/install/buoyancy_plugin/lib/libbuoyancy_plugin.so">
-        <fluid_density>1000</fluid_density>
-        <surface_z>0.0</surface_z>
-        <link name="base_link">
-            <waterplane_area>0.4</waterplane_area>
-            <height>0.2</height>
-            <linear_damping>60.0</linear_damping>
-            <angular_damping>10.0</angular_damping>
-            <k_ righting>50.0</k_righting>
-            <cob>
-            <x>0</x>
-            <y>0</y>
-            <z>-0.05</z>
-            </cob>
-        </link>
-        </plugin>
-    </gazebo>
+<?xml version="1.0"?>
+<robot name="ele306baat" xmlns:xacro="http://www.ros.org/wiki/xacro">
+  <!-- Xacro-parametre (i meter og kg) -->
+    <xacro:property name="m" value="30"/>
+    <xacro:property name="a" value="1.0"/>  <!-- lengde -->
+    <xacro:property name="b" value="0.4"/>  <!-- bredde -->
+    <xacro:property name="c" value="0.2"/>  <!-- høyde -->
+    <xacro:property name="ox" value="0.5"/>  <!-- a/2 -->
+    <xacro:property name="oy" value="-0.2"/>  <!-- b/2 -->
+    <xacro:property name="oz" value="-0.1"/>  <!-- c/2 -->
+  <link name="base_link">
+    <inertial>
+      <origin xyz="0 0 0" rpy="0 0 0"/>
+      <mass value="${m}"/>
+      <inertia
+        ixx="${(1.0/12.0)*m*(b*b + c*c)}"
+        iyy="${(1.0/12.0)*m*(a*a + c*c)}"
+        izz="${(1.0/12.0)*m*(a*a + b*b)}"
+        ixy="0" iyz="0" ixz="0"/>
+    </inertial>
+    <visual name="base_link_visual">
+      <origin xyz="${ox} ${oy} ${oz}" rpy="0 0 0"/>
+      <geometry>
+        <!-- bruk package:// i ROS 2 -->
+        <mesh filename="$(find usv_package)/meshes/base_link.stl" scale="0.001 0.001 0.001"/>
+      </geometry>
+    </visual>
+    <collision name="base_link_collision">
+      <origin xyz="${ox} ${oy} ${oz}" rpy="0 0 0"/>
+      <geometry>
+        <mesh filename="$(find usv_package)/meshes/base_link.stl" scale="0.001 0.001 0.001"/>
+      </geometry>
+    </collision>
+  </link>
+  <!-- Gazebo-tillegg: la Gazebo finne plugin via GAZEBO_PLUGIN_PATH -->
+  <gazebo>
+    <plugin name="buoyancy" filename="libbuoyancy_plugin.so">
+      <fluid_density>1000</fluid_density>
+      <surface_z>0.0</surface_z>
+      <link name="base_link">
+        <waterplane_area>0.4</waterplane_area>
+        <height>0.2</height>
+        <linear_damping>60.0</linear_damping>
+        <angular_damping>10.0</angular_damping>
+        <k_righting>50.0</k_righting>
+        <cob>
+          <x>0</x><y>0</y><z>-0.05</z>
+        </cob>
+      </link>
+    </plugin>
+  </gazebo>
 </robot>

Commit message: lagt til thrustere(ikke fungerende)

File: urdf/ele306baat.urdf.xacro (robot description, xacro)
@@ -9,4 +9,8 @@
     <xacro:property name="oy" value="-0.2"/>  <!-- b/2 -->
     <xacro:property name="oz" value="-0.1"/>  <!-- c/2 -->
+    <xacro:property name="y_off" value="0.22"/>  <!-- avstand sidelengs fra CoM (m) -->
+    <xacro:property name="thr_r" value="0.05"/>  <!-- radius på thruster-visual -->
+    <xacro:property name="thr_l" value="0.06"/>  <!-- lengde på thruster-visual -->
+    <xacro:property name="thr_m" value="0.001"/> <!-- liten masse -->
   <link name="base_link">
     <inertial>
@@ -33,4 +37,49 @@
     </collision>
   </link>
+  <!-- VENSTRE THRUSTER (y>0) -->
+  <link name="thr_left">
+    <inertial>
+      <origin xyz="0 0 0" rpy="0 0 0"/>
+      <mass value="${thr_m}"/>
+      <inertia ixx="1e-6" iyy="1e-6" izz="1e-6" ixy="0" ixz="0" iyz="0"/>
+    </inertial>
+    <visual>
+      <!-- URDF-sylinder peker langs z; roter til x -->
+      <origin xyz="0 0 0" rpy="0 1.57079632679 0"/>
+      <geometry><cylinder radius="${thr_r}" length="${thr_l}"/></geometry>
+      <material name="thr_black"><color rgba="0.1 0.1 0.1 1.0"/></material>
+    </visual>
+    <collision>
+      <origin xyz="0 0 0" rpy="0 1.57079632679 0"/>
+      <geometry><cylinder radius="${thr_r}" length="${thr_l}"/></geometry>
+    </collision>
+  </link>
+  <!-- HØYRE THRUSTER (y<0) -->
+  <link name="thr_right">
+    <inertial>
+      <origin xyz="0 0 0" rpy="0 0 0"/>
+      <mass value="${thr_m}"/>
+      <inertia ixx="1e-6" iyy="1e-6" izz="1e-6" ixy="0" ixz="0" iyz="0"/>
+    </inertial>
+    <visual>
+      <origin xyz="0 0 0" rpy="0 1.57079632679 0"/>
+      <geometry><cylinder radius="${thr_r}" length="${thr_l}"/></geometry>
+      <material name="thr_black"><color rgba="0.1 0.1 0.1 1.0"/></material>
+    </visual>
+    <collision>
+      <origin xyz="0 0 0" rpy="0 1.57079632679 0"/>
+      <geometry><cylinder radius="${thr_r}" length="${thr_l}"/></geometry>
+    </collision>
+  </link>
+  <joint name="thr_left_fixed" type="fixed">
+    <parent link="base_link"/>
+    <child  link="thr_left"/>
+    <origin xyz="0 ${y_off} 0" rpy="0 0 0"/>
+  </joint>
+  <joint name="thr_right_fixed" type="fixed">
+    <parent link="base_link"/>
+    <child  link="thr_right"/>
+    <origin xyz="0 ${-y_off} 0" rpy="0 0 0"/>
+  </joint>
   <!-- Gazebo-tillegg: la Gazebo finne plugin via GAZEBO_PLUGIN_PATH -->
   <gazebo>
@@ -39,5 +88,5 @@
       <surface_z>0.0</surface_z>
       <link name="base_link">
-        <waterplane_area>0.4</waterplane_area>
+        <waterplane_area>1</waterplane_area>
         <height>0.2</height>
         <linear_damping>60.0</linear_damping>
@@ -49,4 +98,20 @@
       </link>
     </plugin>
+    <!-- VENSTRE -->
+    <plugin name="thr_left_force" filename="libgazebo_ros_force.so">
+    <ros>
+      <namespace>/usv</namespace>
+      <remapping>~/force:=/usv/left_thrust</remapping>
+    </ros>
+    <body_name>thr_left</body_name>
+    </plugin>
+    <!-- HØYRE -->
+    <plugin name="thr_right_force" filename="libgazebo_ros_force.so">
+      <ros>
+        <namespace>/usv</namespace>
+        <remapping>~/force:=/usv/right_thrust</remapping>
+      </ros>
+      <body_name>thr_right</body_name>
+    </plugin>
   </gazebo>
 </robot>

Commit message: same

File: urdf/ele306baat.urdf.xacro (robot description, xacro)
@@ -72,16 +72,26 @@
     </collision>
   </link>
-  <joint name="thr_left_fixed" type="fixed">
+  <!-- VENSTRE: yaw rundt z, plassert ved (0, +y_off, 0) -->
+  <joint name="thr_left_yaw" type="revolute">
     <parent link="base_link"/>
     <child  link="thr_left"/>
     <origin xyz="0 ${y_off} 0" rpy="0 0 0"/>
+    <axis xyz="0 0 1"/>                       <!-- yaw-akse -->
+    <limit lower="-1.5708" upper="1.5708" effort="15.0" velocity="2.5"/>
+    <dynamics damping="0.5" friction="0.1"/>
   </joint>
-  <joint name="thr_right_fixed" type="fixed">
+  <!-- HØYRE: yaw rundt z, plassert ved (0, -y_off, 0) -->
+  <joint name="thr_right_yaw" type="revolute">
     <parent link="base_link"/>
     <child  link="thr_right"/>
     <origin xyz="0 ${-y_off} 0" rpy="0 0 0"/>
+    <axis xyz="0 0 1"/>
+    <limit lower="-1.5708" upper="1.5708"
+          effort="15.0" velocity="2.5"/>
+    <dynamics damping="0.5" friction="0.1"/>
   </joint>
   <!-- Gazebo-tillegg: la Gazebo finne plugin via GAZEBO_PLUGIN_PATH -->
   <gazebo>
+    <disableFixedJointLumping>true</disableFixedJointLumping>
     <plugin name="buoyancy" filename="libbuoyancy_plugin.so">
       <fluid_density>1000</fluid_density>
@@ -89,29 +99,45 @@
       <link name="base_link">
         <waterplane_area>1</waterplane_area>
-        <height>0.2</height>
+        <height>0.25</height>
         <linear_damping>60.0</linear_damping>
-        <angular_damping>10.0</angular_damping>
+        <angular_damping>20.0</angular_damping>
         <k_righting>50.0</k_righting>
         <cob>
-          <x>0</x><y>0</y><z>-0.05</z>
+          <x>0</x><y>0</y><z>-0.01</z>
         </cob>
       </link>
     </plugin>
-    <!-- VENSTRE -->
-    <plugin name="thr_left_force" filename="libgazebo_ros_force.so">
+  <plugin name="thr_left_force" filename="libgazebo_ros_force.so">
     <ros>
       <namespace>/usv</namespace>
-      <remapping>~/force:=/usv/left_thrust</remapping>
+      <remapping>gazebo_ros_force:=/usv/left_thrust</remapping>
     </ros>
-    <body_name>thr_left</body_name>
-    </plugin>
-    <!-- HØYRE -->
-    <plugin name="thr_right_force" filename="libgazebo_ros_force.so">
-      <ros>
-        <namespace>/usv</namespace>
-        <remapping>~/force:=/usv/right_thrust</remapping>
-      </ros>
-      <body_name>thr_right</body_name>
-    </plugin>
+    <link_name>thr_left</link_name>
+    <force_frame>link</force_frame>   <!-- kraft i thruster-linkens ramme -->
+  </plugin>
+  <plugin name="thr_right_force" filename="libgazebo_ros_force.so">
+    <ros>
+      <namespace>/usv</namespace>
+      <remapping>gazebo_ros_force:=/usv/right_thrust</remapping>
+    </ros>
+    <link_name>thr_right</link_name>
+    <force_frame>link</force_frame>
+  </plugin>
   </gazebo>
+  <ros2_control name="usv_hw" type="system">
+    <hardware>
+      <plugin>gazebo_ros2_control/DefaultSystem</plugin>
+    </hardware>
+    <!-- Vi styrer yaw-posisjon på begge -->
+    <joint name="thr_left_yaw">
+      <command_interface name="position"/>
+      <state_interface   name="position"/>
+      <state_interface   name="velocity"/>
+    </joint>
+    <joint name="thr_right_yaw">
+      <command_interface name="position"/>
+      <state_interface   name="position"/>
+      <state_interface   name="velocity"/>
+    </joint>
+  </ros2_control>
 </robot>

Commit message: noen tweaks til båt params

File: urdf/ele306baat.urdf.xacro (robot description, xacro)
@@ -15,5 +15,5 @@
   <link name="base_link">
     <inertial>
-      <origin xyz="0 0 0" rpy="0 0 0"/>
+      <origin xyz="0 0 -0.1" rpy="0 0 0"/>
       <mass value="${m}"/>
       <inertia
@@ -76,8 +76,8 @@
     <parent link="base_link"/>
     <child  link="thr_left"/>
-    <origin xyz="0 ${y_off} 0" rpy="0 0 0"/>
+    <origin xyz="0 ${y_off} -0.1" rpy="0 0 0"/>
     <axis xyz="0 0 1"/>                       <!-- yaw-akse -->
     <limit lower="-1.5708" upper="1.5708" effort="15.0" velocity="2.5"/>
-    <dynamics damping="0.5" friction="0.1"/>
+    <dynamics damping="1" friction="10"/>
   </joint>
   <!-- HØYRE: yaw rundt z, plassert ved (0, -y_off, 0) -->
@@ -85,9 +85,9 @@
     <parent link="base_link"/>
     <child  link="thr_right"/>
-    <origin xyz="0 ${-y_off} 0" rpy="0 0 0"/>
+    <origin xyz="0 ${-y_off} -0.1" rpy="0 0 0"/>
     <axis xyz="0 0 1"/>
     <limit lower="-1.5708" upper="1.5708"
           effort="15.0" velocity="2.5"/>
-    <dynamics damping="0.5" friction="0.1"/>
+    <dynamics damping="1" friction="10"/>
   </joint>
   <!-- Gazebo-tillegg: la Gazebo finne plugin via GAZEBO_PLUGIN_PATH -->
@@ -98,11 +98,11 @@
       <surface_z>0.0</surface_z>
       <link name="base_link">
-        <waterplane_area>1</waterplane_area>
-        <height>0.25</height>
-        <linear_damping>60.0</linear_damping>
-        <angular_damping>20.0</angular_damping>
+        <waterplane_area>0.4</waterplane_area>
+        <height>0.2</height>
+        <linear_damping>30.0</linear_damping>
+        <angular_damping>30.0</angular_damping>
         <k_righting>50.0</k_righting>
         <cob>
-          <x>0</x><y>0</y><z>-0.01</z>
+          <x>0</x><y>0</y><z>0.13</z>
         </cob>
       </link>

File: urdf/robot_description.urdf.xacro (robot description, xacro)
@@ -7,5 +7,5 @@
     <inertial>
       <mass value="30.0"/>
-      <origin xyz="0 0 0"/>
+      <origin xyz="0 0 -0.2"/>
       <!-- Boks 1x0.4x0.2 m, m=80 kg, CoM i origo:
            Ixx = 1/12*m*(0.4^2+0.2^2) = 1.3333
@@ -36,12 +36,12 @@
       <link name="DUMMY">
         <waterplane_area>0.4</waterplane_area>
-        <height>0.2</height>
+        <height>0.3</height>
         <linear_damping>60.0</linear_damping>
-        <angular_damping>10.0</angular_damping>
+        <angular_damping>15.0</angular_damping>
         <k_righting>50.0</k_righting>
         <cob>
           <x>0</x>
           <y>0</y>
-          <z>-0.05</z>
+          <z>-0.01</z>
         </cob>
       </link>
