Commit message: ??

File: install/usv_package/share/usv_package/urdf/ele306baat.urdf.xacro (robot description, xacro)
@@ -9,4 +9,8 @@
     <xacro:property name="oy" value="-0.2"/>  <!-- b/2 -->
     <xacro:property name="oz" value="-0.1"/>  <!-- c/2 -->
+    <xacro:property name="y_off" value="0.22"/>  <!-- avstand sidelengs fra CoM (m) -->
+    <xacro:property name="thr_r" value="0.05"/>  <!-- radius på thruster-visual -->
+    <xacro:property name="thr_l" value="0.06"/>  <!-- lengde på thruster-visual -->
+    <xacro:property name="thr_m" value="0.001"/> <!-- liten masse -->
   <link name="base_link">
     <inertial>
@@ -33,20 +37,107 @@
     </collision>
   </link>
+  <!-- VENSTRE THRUSTER (y>0) -->
+  <link name="thr_left">
+    <inertial>
+      <origin xyz="0 0 0" rpy="0 0 0"/>
+      <mass value="${thr_m}"/>
+      <inertia ixx="1e-6" iyy="1e-6" izz="1e-6" ixy="0" ixz="0" iyz="0"/>
+    </inertial>
+    <visual>
+      <!-- URDF-sylinder peker langs z; roter til x -->
+      <origin xyz="0 0 0" rpy="0 1.57079632679 0"/>
+      <geometry><cylinder radius="${thr_r}" length="${thr_l}"/></geometry>
+      <material name="thr_black"><color rgba="0.1 0.1 0.1 1.0"/></material>
+    </visual>
+    <collision>
+      <origin xyz="0 0 0" rpy="0 1.57079632679 0"/>
+      <geometry><cylinder radius="${thr_r}" length="${thr_l}"/></geometry>
+    </collision>
+  </link>
+  <!-- HØYRE THRUSTER (y<0) -->
+  <link name="thr_right">
+    <inertial>
+      <origin xyz="0 0 0" rpy="0 0 0"/>
+      <mass value="${thr_m}"/>
+      <inertia ixx="1e-6" iyy="1e-6" izz="1e-6" ixy="0" ixz="0" iyz="0"/>
+    </inertial>
+    <visual>
+      <origin xyz="0 0 0" rpy="0 1.57079632679 0"/>
+      <geometry><cylinder radius="${thr_r}" length="${thr_l}"/></geometry>
+      <material name="thr_black"><color rgba="0.1 0.1 0.1 1.0"/></material>
+    </visual>
+    <collision>
+      <origin xyz="0 0 0" rpy="0 1.57079632679 0"/>
+      <geometry><cylinder radius="${thr_r}" length="${thr_l}"/></geometry>
+    </collision>
+  </link>
+  <!-- VENSTRE: yaw rundt z, plassert ved (0, +y_off, 0) -->
+  <joint name="thr_left_yaw" type="revolute">
+    <parent link="base_link"/>
+    <child  link="thr_left"/>
+    <origin xyz="0 ${y_off} 0" rpy="0 0 0"/>
+    <axis xyz="0 0 1"/>                       <!-- yaw-akse -->
+    <limit lower="-1.5708" upper="1.5708" effort="15.0" velocity="2.5"/>
+    <dynamics damping="0.5" friction="0.1"/>
+  </joint>
+  <!-- HØYRE: yaw rundt z, plassert ved (0, -y_off, 0) -->
+  <joint name="thr_right_yaw" type="revolute">
+    <parent link="base_link"/>
+    <child  link="thr_right"/>
+    <origin xyz="0 ${-y_off} 0" rpy="0 0 0"/>
+    <axis xyz="0 0 1"/>
+    <limit lower="-1.5708" upper="1.5708"
+          effort="15.0" velocity="2.5"/>
+    <dynamics damping="0.5" friction="0.1"/>
+  </joint>
   <!-- Gazebo-tillegg: la Gazebo finne plugin via GAZEBO_PLUGIN_PATH -->
   <gazebo>
+    <disableFixedJointLumping>true</disableFixedJointLumping>
     <plugin name="buoyancy" filename="libbuoyancy_plugin.so">
       <fluid_density>1000</fluid_density>
       <surface_z>0.0</surface_z>
       <link name="base_link">
-        <waterplane_area>0.4</waterplane_area>
-        <height>0.2</height>
+        <waterplane_area>1</waterplane_area>
+        <height>0.25</height>
         <linear_damping>60.0</linear_damping>
-        <angular_damping>10.0</angular_damping>
+        <angular_damping>20.0</angular_damping>
         <k_righting>50.0</k_righting>
         <cob>
-          <x>0</x><y>0</y><z>-0.05</z>
+          <x>0</x><y>0</y><z>-0.01</z>
         </cob>
       </link>
     </plugin>
+  <plugin name="thr_left_force" filename="libgazebo_ros_force.so">
+    <ros>
+      <namespace>/usv</namespace>
+      <remapping>gazebo_ros_force:=/usv/left_thrust</remapping>
+    </ros>
+    <link_name>thr_left</link_name>
+    <force_frame>link</force_frame>   <!-- kraft i thruster-linkens ramme -->
+  </plugin>
+  <plugin name="thr_right_force" filename="libgazebo_ros_force.so">
+    <ros>
+      <namespace>/usv</namespace>
+      <remapping>gazebo_ros_force:=/usv/right_thrust</remapping>
+    </ros>
+    <link_name>thr_right</link_name>
+    <force_frame>link</force_frame>
+  </plugin>
   </gazebo>
+  <ros2_control name="usv_hw" type="system">
+    <hardware>
+      <plugin>gazebo_ros2_control/DefaultSystem</plugin>
+    </hardware>
+    <!-- Vi styrer yaw-posisjon på begge -->
+    <joint name="thr_left_yaw">
+      <command_interface name="position"/>
+      <state_interface   name="position"/>
+      <state_interface   name="velocity"/>
+    </joint>
+    <joint name="thr_right_yaw">
+      <command_interface name="position"/>
+      <state_interface   name="position"/>
+      <state_interface   name="velocity"/>
+    </joint>
+  </ros2_control>
 </robot>
