Commit message: for editing

File: urdf/URDFEDIT/ele306baat_V2.urdf.xacro (robot description, xacro)
@@ -28,5 +28,5 @@
       <geometry>
         <!-- bruk package:// i ROS 2 etter hvert -->
-        <mesh filename="$(find usv_package)/meshes/base_link.stl" scale="0.001 0.001 0.001"/>
+        <mesh filename="base_link.stl" scale="0.001 0.001 0.001"/>
       </geometry>
     </visual>
@@ -34,5 +34,5 @@
       <origin xyz="${ox} ${oy} ${oz}" rpy="0 0 0"/>
       <geometry>
-        <mesh filename="$(find usv_package)/meshes/base_link.stl" scale="0.001 0.001 0.001"/>
+        <mesh filename="base_link.stl" scale="0.001 0.001 0.001"/>
       </geometry>
     </collision>
@@ -116,5 +116,5 @@
       <origin xyz="0.0 0.0 0.0" rpy="0.0 0.0 0.0"/>
       <geometry>
-        <mesh filename="$(find usv_package)/meshes/5DOF_V2-v1_Base-v1.stl" scale="0.001 0.001 0.001"/>
+        <mesh filename="5DOF_V2-v1_Base-v1.stl" scale="0.001 0.001 0.001"/>
       </geometry>
     </visual>
@@ -122,5 +122,5 @@
       <origin xyz="0.0 0.0 0.0" rpy="0.0 0.0 0.0"/>
       <geometry>
-        <mesh filename="$(find usv_package)/meshes/5DOF_V2-v1_Base-v1.stl" scale="0.001 0.001 0.001"/>
+        <mesh filename="5DOF_V2-v1_Base-v1.stl" scale="0.001 0.001 0.001"/>
       </geometry>
     </collision>
@@ -136,5 +136,5 @@
       <origin xyz="0.0 0.0 0.0" rpy="0.0 0.0 0.0"/>
       <geometry>
-        <mesh filename="$(find usv_package)/meshes/5DOF_V2-v1_Base_tube2-v1.stl" scale="0.001 0.001 0.001"/>
+        <mesh filename="5DOF_V2-v1_Base_tube2-v1.stl" scale="0.001 0.001 0.001"/>
       </geometry>
     </visual>
@@ -142,5 +142,5 @@
       <origin xyz="0.0 0.0 0.0" rpy="0.0 0.0 0.0"/>
       <geometry>
-        <mesh filename="$(find usv_package)/meshes/5DOF_V2-v1_Base_tube2-v1.stl" scale="0.001 0.001 0.001"/>
+        <mesh filename="5DOF_V2-v1_Base_tube2-v1.stl" scale="0.001 0.001 0.001"/>
       </geometry>
     </collision>
@@ -156,5 +156,5 @@
       <origin xyz="0.0 0.0 0.0" rpy="0.0 0.0 0.0"/>
       <geometry>
-        <mesh filename="$(find usv_package)/meshes/5DOF_V2-v1_Base_tube-v1.stl" scale="0.001 0.001 0.001"/>
+        <mesh filename="5DOF_V2-v1_Base_tube-v1.stl" scale="0.001 0.001 0.001"/>
       </geometry>
     </visual>
@@ -162,5 +162,5 @@
       <origin xyz="0.0 0.0 0.0" rpy="0.0 0.0 0.0"/>
       <geometry>
-        <mesh filename="$(find usv_package)/meshes/5DOF_V2-v1_Base_tube-v1.stl" scale="0.001 0.001 0.001"/>
+        <mesh filename="5DOF_V2-v1_Base_tube-v1.stl" scale="0.001 0.001 0.001"/>
       </geometry>
     </collision>
@@ -176,5 +176,5 @@
       <origin xyz="0.0 0.0 0.0" rpy="0.0 0.0 0.0"/>
       <geometry>
-        <mesh filename="$(find usv_package)/meshes/5DOF_V2-v1_Ledd1-v1.stl" scale="0.001 0.001 0.001"/>
+        <mesh filename="5DOF_V2-v1_Ledd1-v1.stl" scale="0.001 0.001 0.001"/>
       </geometry>
     </visual>
@@ -182,5 +182,5 @@
       <origin xyz="0.0 0.0 0.0" rpy="0.0 0.0 0.0"/>
       <geometry>
-        <mesh filename="$(find usv_package)/meshes/5DOF_V2-v1_Ledd1-v1.stl" scale="0.001 0.001 0.001"/>
+        <mesh filename="5DOF_V2-v1_Ledd1-v1.stl" scale="0.001 0.001 0.001"/>
       </geometry>
     </collision>
@@ -196,5 +196,5 @@
       <origin xyz="0.0 0.0 0.0" rpy="0.0 0.0 0.0"/>
       <geometry>
-        <mesh filename="$(find usv_package)/meshes/5DOF_V2-v1_Ledd2-v1.stl" scale="0.001 0.001 0.001"/>
+        <mesh filename="5DOF_V2-v1_Ledd2-v1.stl" scale="0.001 0.001 0.001"/>
       </geometry>
     </visual>
@@ -202,5 +202,5 @@
       <origin xyz="0.0 0.0 0.0" rpy="0.0 0.0 0.0"/>
       <geometry>
-        <mesh filename="$(find usv_package)/meshes/5DOF_V2-v1_Ledd2-v1.stl" scale="0.001 0.001 0.001"/>
+        <mesh filename="5DOF_V2-v1_Ledd2-v1.stl" scale="0.001 0.001 0.001"/>
       </geometry>
     </collision>
@@ -216,5 +216,5 @@
       <origin xyz="0.0 0.0 0.0" rpy="0.0 0.0 0.0"/>
       <geometry>
-        <mesh filename="$(find usv_package)/meshes/5DOF_V2-v1_Ledd-4-v1.stl" scale="0.001 0.001 0.001"/>
+        <mesh filename="5DOF_V2-v1_Ledd-4-v1.stl" scale="0.001 0.001 0.001"/>
       </geometry>
     </visual>
@@ -222,5 +222,5 @@
       <origin xyz="0.0 0.0 0.0" rpy="0.0 0.0 0.0"/>
       <geometry>
-        <mesh filename="$(find usv_package)/meshes/5DOF_V2-v1_Ledd-4-v1.stl" scale="0.001 0.001 0.001"/>
+        <mesh filename="5DOF_V2-v1_Ledd-4-v1.stl" scale="0.001 0.001 0.001"/>
       </geometry>
     </collision>
@@ -236,5 +236,5 @@
       <origin xyz="0.0 0.0 0.0" rpy="0.0 0.0 0.0"/>
       <geometry>
-        <mesh filename="$(find usv_package)/meshes/5DOF_V2-v1_fryer-complete-v1.stl" scale="0.001 0.001 0.001"/>
+        <mesh filename="5DOF_V2-v1_fryer-complete-v1.stl" scale="0.001 0.001 0.001"/>
       </geometry>
     </visual>
@@ -242,5 +242,5 @@
       <origin xyz="0.0 0.0 0.0" rpy="0.0 0.0 0.0"/>
       <geometry>
-        <mesh filename="$(find usv_package)/meshes/5DOF_V2-v1_fryer-complete-v1.stl" scale="0.001 0.001 0.001"/>
+        <mesh filename="5DOF_V2-v1_fryer-complete-v1.stl" scale="0.001 0.001 0.001"/>
       </geometry>
     </collision>
@@ -256,5 +256,5 @@
       <origin xyz="0.0 0.0 0.0" rpy="0.0 0.0 0.0"/>
       <geometry>
-        <mesh filename="$(find usv_package)/meshes/5DOF_V2-v1_Ledd5-v1.stl" scale="0.001 0.001 0.001"/>
+        <mesh filename="5DOF_V2-v1_Ledd5-v1.stl" scale="0.001 0.001 0.001"/>
       </geometry>
     </visual>
@@ -263,5 +263,5 @@
       <geometry>
         <!-- FIKSET: fjernet dobbel $(find usv_package)/ -->
-        <mesh filename="$(find usv_package)/meshes/5DOF_V2-v1_Ledd5-v1.stl" scale="0.001 0.001 0.001"/>
+        <mesh filename="5DOF_V2-v1_Ledd5-v1.stl" scale="0.001 0.001 0.001"/>
       </geometry>
     </collision>

Commit message: fiksa arm

File: urdf/URDFEDIT/ele306baat_V2.urdf.xacro (robot description, xacro)
@@ -45,14 +45,4 @@
       <inertia ixx="1e-6" iyy="1e-6" izz="1e-6" ixy="0" ixz="0" iyz="0"/>
     </inertial>
-    <visual>
-      <!-- URDF-sylinder peker langs z; roter til x -->
-      <origin xyz="0 0 0" rpy="0 1.57079632679 0"/>
-      <geometry>
-        <cylinder radius="${thr_r}" length="${thr_l}"/>
-      </geometry>
-      <material name="thr_black">
-        <color rgba="0.1 0.1 0.1 1.0"/>
-      </material>
-    </visual>
     <collision>
       <origin xyz="0 0 0" rpy="0 1.57079632679 0"/>
@@ -69,13 +59,4 @@
       <inertia ixx="1e-6" iyy="1e-6" izz="1e-6" ixy="0" ixz="0" iyz="0"/>
     </inertial>
-    <visual>
-      <origin xyz="0 0 0" rpy="0 1.57079632679 0"/>
-      <geometry>
-        <cylinder radius="${thr_r}" length="${thr_l}"/>
-      </geometry>
-      <material name="thr_black">
-        <color rgba="0.1 0.1 0.1 1.0"/>
-      </material>
-    </visual>
     <collision>
       <origin xyz="0 0 0" rpy="0 1.57079632679 0"/>
@@ -89,5 +70,5 @@
     <parent link="base_link"/>
     <child  link="thr_left"/>
-    <origin xyz="0 ${y_off} -0.1" rpy="0 0 0"/>
+    <origin xyz="0 ${y_off} -0.08" rpy="0 0 0"/>
     <axis xyz="0 0 1"/>                       <!-- yaw-akse -->
     <limit lower="-1.5708" upper="1.5708" effort="15.0" velocity="2.5"/>
@@ -98,5 +79,5 @@
     <parent link="base_link"/>
     <child  link="thr_right"/>
-    <origin xyz="0 ${-y_off} -0.1" rpy="0 0 0"/>
+    <origin xyz="0 ${-y_off} -0.08" rpy="0 0 0"/>
     <axis xyz="0 0 1"/>
     <limit lower="-1.5708" upper="1.5708" effort="15.0" velocity="2.5"/>
@@ -174,5 +155,5 @@
     </inertial>
     <visual name="5DOF_V2-v1_Ledd1-v1_visual">
-      <origin xyz="0.0 0.0 0.0" rpy="0.0 0.0 0.0"/>
+      <origin xyz="0.0 -0.03 0.0" rpy="0.0 0.0 0.0"/>
       <geometry>
         <mesh filename="5DOF_V2-v1_Ledd1-v1.stl" scale="0.001 0.001 0.001"/>
@@ -194,5 +175,5 @@
     </inertial>
     <visual name="5DOF_V2-v1_Ledd2-v1_visual">
-      <origin xyz="0.0 0.0 0.0" rpy="0.0 0.0 0.0"/>
+      <origin xyz="0.0 -0.03 0.0" rpy="0.0 0.0 0.0"/>
       <geometry>
         <mesh filename="5DOF_V2-v1_Ledd2-v1.stl" scale="0.001 0.001 0.001"/>
@@ -200,5 +181,5 @@
     </visual>
     <collision name="5DOF_V2-v1_Ledd2-v1_collision">
-      <origin xyz="0.0 0.0 0.0" rpy="0.0 0.0 0.0"/>
+      <origin xyz="0.0 -0.03 0.0" rpy="0.0 0.0 0.0"/>
       <geometry>
         <mesh filename="5DOF_V2-v1_Ledd2-v1.stl" scale="0.001 0.001 0.001"/>
@@ -214,5 +195,5 @@
     </inertial>
     <visual name="5DOF_V2-v1_Ledd-4-v1_visual">
-      <origin xyz="0.0 0.0 0.0" rpy="0.0 0.0 0.0"/>
+      <origin xyz="-0.02 0.02 -0.02" rpy="1.5708 0.0 0.0"/>
       <geometry>
         <mesh filename="5DOF_V2-v1_Ledd-4-v1.stl" scale="0.001 0.001 0.001"/>
@@ -220,5 +201,5 @@
     </visual>
     <collision name="5DOF_V2-v1_Ledd-4-v1_collision">
-      <origin xyz="0.0 0.0 0.0" rpy="0.0 0.0 0.0"/>
+      <origin xyz="0.0 0.0 0.0" rpy="1.5708 0.0 0.0"/>
       <geometry>
         <mesh filename="5DOF_V2-v1_Ledd-4-v1.stl" scale="0.001 0.001 0.001"/>
@@ -289,5 +270,5 @@
   </joint>
   <joint name="5DOF_V2-v1_Base_tube-v1_Revolute-13" type="continuous">
-    <origin xyz="0 -0.03 0.08"
+    <origin xyz="0. 0 0.12"
             rpy="0 3.14 1.5708"/>
     <parent link="5DOF_V2-v1_Base_tube-v1"/>
@@ -296,29 +277,29 @@
   </joint>
   <joint name="5DOF_V2-v1_Ledd1-v1_Revolute-4" type="continuous">
-    <origin xyz="-9.16609224077547e-10 0.37999999999999307 0.07499999504391575"
-            rpy="-1.5707963267948963 0.012632873265397596 1.5708"/>
+    <origin xyz="0 0.35 0.1"
+            rpy="0 3.14 0"/>
     <parent link="5DOF_V2-v1_Ledd1-v1"/>
     <child  link="5DOF_V2-v1_Ledd2-v1"/>
-    <axis xyz="-0.012633000000000004 -0.99992 -5.799401443819225e-33"/>
+    <axis xyz="0 0 1"/>
   </joint>
   <joint name="5DOF_V2-v1_Ledd-4-v1_Revolute-9" type="continuous">
-    <origin xyz="0.020000001123706285 0.039999999999984936 0.019999999181395153"
-            rpy="-3.1415926535897927 0.0126328732654071 -2.226143245893908e-15"/>
+    <origin xyz="-0.0 0 0.02"
+            rpy="0 0 0"/>
     <parent link="5DOF_V2-v1_Ledd-4-v1"/>
     <child  link="5DOF_V2-v1_Ledd5-v1"/>
-    <axis xyz="-1.7347234759758815e-18 -1.0 0.0"/>
+    <axis xyz="0 0 1.0"/>
   </joint>
   <joint name="5DOF_V2-v1_Ledd5-v1_Rigid-11" type="fixed">
-    <origin xyz="8.18604810604029e-10 1.1237057151447515e-09 1.3926637620897963e-14"
-            rpy="7.95274871898862e-16 2.5014215493744513e-14 1.5581634535294897"/>
+    <origin xyz="-0.012 0 0.1716"
+            rpy="1.5708 1.5708 0"/>
     <parent link="5DOF_V2-v1_Ledd5-v1"/>
     <child  link="5DOF_V2-v1_fryer-complete-v1"/>
   </joint>
   <joint name="5DOF_V2-v1_Ledd2-v1_Revolute-15" type="continuous">
-    <origin xyz="3.8774454111489834e-07 0.3299999999999883 0.07499999975316342"
+    <origin xyz="0 0.3 0.07"
             rpy="1.570796326794897 -0.012632873265408419 -3.1415926535897913"/>
     <parent link="5DOF_V2-v1_Ledd2-v1"/>
     <child  link="5DOF_V2-v1_Ledd-4-v1"/>
-    <axis xyz="0.012633 0.99992 2.3493747465131305e-32"/>
+    <axis xyz="0 1 0"/>
   </joint>
   <!-- ============================ -->
